Commit message: Cambios actuales para stalker3000

File: src/el5206_description/urdf/turtlebot3_burger.gazebo.xacro (robot description, xacro)
@@ -136,3 +136,45 @@
     </sensor>
   </gazebo>
+<gazebo reference="depth_camera">
+    <sensor name="depth_camera_camera" type="depth">
+      <always_on>true</always_on>
+    <update_rate>1</update_rate>
+    <camera>
+      <horizontal_fov>1.047198</horizontal_fov>
+      <image>
+        <width>640</width>
+        <height>480</height>
+        <format>R8G8B8</format>
+      </image>
+      <clip>
+        <near>0.05</near>
+        <far>3</far>
+      </clip>
+    </camera>
+    <plugin name="depth_camera_controller" filename="libgazebo_ros_openni_kinect.so">
+      <baseline>0.2</baseline>
+      <alwaysOn>true</alwaysOn>
+      <updateRate>0.0</updateRate>
+      <cameraName>camera_ir</cameraName>
+      <imageTopicName>camera/color/image_raw</imageTopicName>
+      <cameraInfoTopicName>camera/color/camera_info</cameraInfoTopicName>
+      <depthImageTopicName>camera/depth/image_raw</depthImageTopicName>
+      <depthImageInfoTopicName>camera/depth/camera_info</depthImageInfoTopicName>
+      <pointCloudTopicName>camera/depth/points</pointCloudTopicName>
+      <frameName>camera</frameName>
+      <pointCloudCutoff>0.5</pointCloudCutoff>
+      <pointCloudCutoffMax>3.0</pointCloudCutoffMax>
+      <distortionK1>0.00000001</distortionK1>
+      <distortionK2>0.00000001</distortionK2>
+      <distortionK3>0.00000001</distortionK3>
+      <distortionT1>0.00000001</distortionT1>
+      <distortionT2>0.00000001</distortionT2>
+      <CxPrime>0</CxPrime>
+      <Cx>0</Cx>
+      <Cy>0</Cy>
+      <focalLength>0</focalLength>
+      <hackBaseline>0</hackBaseline>
+    </plugin>
+  </sensor>
+</gazebo>
 </robot>

File: src/el5206_description/urdf/turtlebot3_burger.urdf.xacro (robot description, xacro)
@@ -3,4 +3,5 @@
   <xacro:include filename="$(find el5206_description)/urdf/common_properties.xacro"/>
   <xacro:include filename="$(find el5206_description)/urdf/turtlebot3_burger.gazebo.xacro"/>
+  <xacro:property name="camera_link" value="0.05" /> <!-- Size of square 'camera' box -->
   <link name="base_footprint"/>
   <joint name="base_joint" type="fixed">
@@ -140,3 +141,30 @@
     </inertial>
   </link>
+  <joint name="camera_rgb_joint" type="fixed">
+    <origin xyz="0.003 0.011 0.1" rpy="0 0 0"/>
+    <parent link="base_link"/>
+    <child link="depth_camera"/>
+  </joint>
+  <link name="depth_camera">
+    <inertial><mass value="0.1" />
+      <inertia ixx="0.001" ixy="0.0" ixz="0.0"
+               iyy="0.001" iyz="0.0"
+               izz="0.001" /></inertial>
+    <collision name="collision">
+      <geometry>
+        <box size="0.073000 0.276000 0.072000" />
+      </geometry>
+    </collision>
+      <visual name="visual">
+        <geometry>
+          <mesh filename="model://kinect/meshes/kinect.dae" />
+        </geometry>
+      </visual>
+  </link>
+  <joint name="camera_rgb_optical_joint" type="fixed">
+    <origin xyz="0 0 0" rpy="-1.57 0 -1.57"/>
+    <parent link="depth_camera"/>
+    <child link="camera_rgb_optical_frame"/>
+  </joint>
+  <link name="camera_rgb_optical_frame"/>
 </robot>
